File: big-board.kicad_pcb (KiCad board)
At the start: 2 copper layers, 133 parts, among them SW1 SW_Push, SW10 SW_Push, SW11 SW_Push, SW12 SW_Push, SW13 SW_Push, SW14 SW_Push, SW15 SW_Push, SW16 SW_Push, SW17 SW_Push, SW18 SW_Push, SW19 SW_Push, SW2 SW_Push, SW20 SW_Push, SW21 SW_Push, SW22 SW_Push, SW23 SW_Push, SW24 SW_Push, SW25 SW_Push, SW26 SW_Push, SW27 SW_Push, SW28 SW_Push, SW29 SW_Push, SW3 SW_Push, SW30 SW_Push, SW31 SW_Push, SW32 SW_Push, SW33 SW_Push, SW34 SW_Push, SW35 SW_Push, SW36 SW_Push, SW37 SW_Push, SW38 SW_Push, SW39 SW_Push, SW4 SW_Push, SW40 SW_Push, SW41 SW_Push, SW42 SW_Push, SW43 SW_Push, SW44 SW_Push, SW45 SW_Push, SW46 SW_Push, SW47 SW_Push, SW48 SW_Push, SW49 SW_Push, SW5 SW_Push, SW50 SW_Push, SW51 SW_Push, SW52 SW_Push, SW53 SW_Push, SW54 SW_Push, SW55 SW_Push, SW56 SW_Push, SW57 SW_Push, SW58 SW_Push, SW59 SW_Push, SW6 SW_Push, SW60 SW_Push, SW61 SW_Push, SW62 SW_Push, SW63 SW_Push, SW64 SW_Push, SW65 SW_Push, SW66 SW_Push, SW7 SW_Push, SW8 SW_Push, SW9 SW_Push, U1 Pico

Commit message: keep routing
Parts:
- D1, D10, D11, D12, D13, D14, D15, D16, D17, D18, D19, D2, D20, D21, D22, D23, D24, D25, D26, D27, D28, D29, D3, D30, D31, D32, D33, D34, D35, D36, D37, D38, D39, D4, D40, D41, D42, D43, D44, D45, D46, D47, D48, D49, D5, D50, D51, D52, D53, D54, D55, D56, D57, D58, D59, D6, D60, D61, D62, D63, D64, D65, D66, D7, D8, D9: footprint Diode_THT:D_DO-35_SOD27_P2.54mm_Vertical_AnodeUp -> Diode_THT:D_DO-35_SOD27_P7.62mm_Horizontal
- moved D59 6.43 mm to (114.2, 228.0)
- moved D32 6.43 mm to (102.3, 189.9)
- moved D4 6.43 mm to (126.2, 151.8)
- moved D57 6.43 mm to (71.4, 228.0)
- moved D58 6.43 mm to (92.8, 228.0)
- moved D60 6.43 mm to (185.7, 228.0)
- moved D62 6.43 mm to (280.9, 228.0)
- moved D63 6.43 mm to (304.7, 228.0)
- moved D64 6.43 mm to (326.2, 228.0)
- moved D65 6.43 mm to (345.2, 228.0)
- moved D66 6.43 mm to (364.3, 228.0)
- moved D1 6.43 mm to (88.0, 151.8)
- moved D10 6.43 mm to (240.4, 151.8)
- moved D11 6.43 mm to (259.5, 151.8)
- moved D12 6.43 mm to (278.6, 151.8)
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Routing:
- net ROW1: track 58.6 -> 356.1 mm
- net ROW2: track 67.8 -> 321.0 mm
- net ROW0: track 326.3 -> 347.8 mm
- net Net-(D14-A): track 7.73 -> 14.7 mm
- net Net-(D55-A): track 0.00 -> 6.95 mm
- net Net-(D41-A): track 0.00 -> 6.95 mm
- net Net-(D25-A): track 0.00 -> 6.95 mm
- net Net-(D23-A): track 0.00 -> 6.95 mm
- net Net-(D20-A): track 0.00 -> 6.95 mm
- net Net-(D18-A): track 0.00 -> 6.95 mm
- net Net-(D17-A): track 0.00 -> 6.95 mm
- net Net-(D16-A): track 0.00 -> 6.95 mm
- net Net-(D24-A): track 0.00 -> 6.95 mm
- net Net-(D21-A): track 0.00 -> 6.95 mm
- net Net-(D19-A): track 0.00 -> 6.95 mm
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
Commit message: more pcb routing
Parts:
- moved D22 32.3 mm to (206.7, 141.7)
- moved D26 32.3 mm to (282.9, 141.7)
- moved D27 32.3 mm to (301.9, 141.7)
- moved D28 32.3 mm to (321.0, 141.7)
- moved D29 32.3 mm to (344.8, 141.7)
- moved D30 32.3 mm to (378.1, 141.7)
- moved D16 32.3 mm to (87.6, 141.7)
- moved D17 32.3 mm to (111.4, 141.7)
- moved D18 32.3 mm to (130.5, 141.7)
- moved D19 32.3 mm to (149.5, 141.7)
- moved D20 32.3 mm to (168.6, 141.7)
- moved D21 32.3 mm to (187.6, 141.7)
- moved D23 32.3 mm to (225.7, 141.7)
- moved D24 32.3 mm to (244.8, 141.7)
- moved D25 32.3 mm to (263.8, 141.7)
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Connections:
- U1 pad 13: GND -> unconnected-(U1-GND-Pad13)
- U1 pad 18: GND -> unconnected-(U1-GND-Pad18)
- U1 pad 28: GND -> unconnected-(U1-GND-Pad28)
- U1 pad 3: GND -> unconnected-(U1-GND-Pad3)
- U1 pad 33: GNDA -> unconnected-(U1-AGND-Pad33)
- U1 pad 38: GND -> unconnected-(U1-GND-Pad38)
- U1 pad 42: GND -> unconnected-(U1-GND-Pad42)
- U1 pad 8: GND -> unconnected-(U1-GND-Pad8)
Routing:
- net COL5: track 0.00 -> 477.0 mm, vias 0 -> 1
- net COL4: track 0.00 -> 450.2 mm, vias 0 -> 2
- net COL3: track 0.00 -> 228.8 mm
- net COL2: track 0.00 -> 222.7 mm
- net COL1: track 3.25 -> 208.4 mm, vias 0 -> 1
- net COL9: track 0.00 -> 197.3 mm
- net COL7: track 0.00 -> 180.1 mm
- net COL8: track 0.00 -> 178.4 mm
- net COL6: track 0.00 -> 175.7 mm
- net COL0: track 85.1 -> 184.7 mm
- net COL12: track 0.00 -> 80.0 mm
- net COL11: track 0.00 -> 75.7 mm
- net COL10: track 0.00 -> 67.0 mm
- net COL13: track 0.00 -> 21.0 mm
- net Net-(D14-A): track 14.7 -> 6.95 mm
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Other:
- board outline added: 357.2 x 102.4 mm

Commit message: hole
Routing:
- net COL8: track 178.4 -> 414.6 mm
- net COL9: track 197.3 -> 429.5 mm, vias 0 -> 3
- net COL6: track 175.7 -> 363.0 mm
- net COL7: track 180.1 -> 358.2 mm, vias 0 -> 4
Other:
- board size 357.2 x 102.4 mm -> 357.2 x 100 mm

Commit message: finish pcb
Routing:
- net COL14: track 19.0 -> 337.6 mm, vias 0 -> 5
- net COL13: track 21.0 -> 316.2 mm, vias 0 -> 3
- net COL11: track 75.7 -> 356.9 mm, vias 0 -> 2
- net COL12: track 80.0 -> 359.8 mm, vias 0 -> 3
- net COL10: track 67.0 -> 321.3 mm, vias 0 -> 2
Other:
- outline, holes or cut-outs redrawn

Commit message: silkscreen stuff
Parts:
- SW1, SW10, SW11, SW12, SW13, SW15, SW17, SW18, SW19, SW2, SW20, SW21, SW22, SW23, SW24, SW25, SW26, SW27, SW28, SW3, SW30, SW32, SW33, SW34, SW35, SW36, SW37, SW38, SW39, SW4, SW40, SW41, SW42, SW45, SW46, SW47, SW48, SW49, SW5, SW50, SW51, SW52, SW53, SW54, SW56, SW58, SW6, SW64, SW65, SW66, SW7, SW8, SW9: footprint MX_Solderable:MX-Solderable-1U -> 3d:MX-Solderable-1U
Other:
- outline, holes or cut-outs redrawn

Commit message: finish pcb
Routing:
- added copper zone on B.Cu, net GND
- added copper zone on F.Cu, net GND
Other:
- board text added: "keyboard"

Commit message: fix pcb and generate 3d model
Other:
- outline, holes or cut-outs redrawn
Changed lines of the file:
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@@
 		)
 		(embedded_fonts no)
+		(model "${KIPRJMOD}/libraries/Cherry MX.STEP"
+			(offset
+				(xyz 0 1 1.5)
+			)
+			(scale
+				(xyz 1 1 1)
+			)
+			(rotate
+				(xyz -90 -0 -0)
+			)
+		)
 	)
 	(footprint "MX_Solderable:MX-Solderable-1.5U"
@@
 		)
 		(embedded_fonts no)
+		(model "${KIPRJMOD}/libraries/Cherry MX.STEP"
+			(offset
+				(xyz 0 1 1.5)
+			)
+			(scale
+				(xyz 1 1 1)
+			)
+			(rotate
+				(xyz -90 -0 -0)
+			)
+		)
 	)
 	(footprint "3d:MX-Solderable-1U"
@@
 		)
 		(embedded_fonts no)
+		(model "${KIPRJMOD}/libraries/Cherry MX.STEP"
+			(offset
+				(xyz 0 1 1.5)
+			)
+			(scale
+				(xyz 1 1 1)
+			)
+			(rotate
+				(xyz -90 -0 -0)
+			)
+		)
 	)
 	(footprint "3d:MX-Solderable-1U"
@@
 		)
 		(embedded_fonts no)
+		(model "${KIPRJMOD}/libraries/Cherry MX.STEP"
+			(offset
+				(xyz 0 1 1.5)
+			)
+			(scale
+				(xyz 1 1 1)
+			)
+			(rotate
+				(xyz -90 -0 -0)
+			)
+		)
 	)
 	(footprint "3d:MX-Solderable-1U"
@@
 		)
 		(embedded_fonts no)
+		(model "${KIPRJMOD}/libraries/Cherry MX.STEP"
+			(offset
+				(xyz 0 1 1.5)
+			)
+			(scale
+				(xyz 1 1 1)
+			)
+			(rotate
+				(xyz -90 -0 -0)
+			)
+		)
 	)
 	(footprint "3d:MX-Solderable-1U"
@@
 		)
 		(embedded_fonts no)
+		(model "${KIPRJMOD}/libraries/Cherry MX.STEP"
+			(offset
+				(xyz 0 1 1.5)
+			)
+			(scale
+				(xyz 1 1 1)
+			)
+			(rotate
+				(xyz -90 -0 -0)
+			)
+		)
 	)
 	(footprint "3d:MX-Solderable-1U"
@@
 		)
 		(embedded_fonts no)
+		(model "${KIPRJMOD}/libraries/Cherry MX.STEP"
+			(offset
+				(xyz 0 1 1.5)
+			)
+			(scale
+				(xyz 1 1 1)
+			)
+			(rotate
+				(xyz -90 -0 -0)
+			)
+		)
 	)
 	(footprint "MX_Solderable:MX-Solderable-2.25U"
@@
 		)
 		(embedded_fonts no)
+		(model "${KIPRJMOD}/libraries/Cherry MX.STEP"
+			(offset
+				(xyz 0 1 1.5)
+			)
+			(scale
+				(xyz 1 1 1)
+			)
+			(rotate
+				(xyz -90 -0 -0)
+			)
+		)
 	)
 	(footprint "3d:MX-Solderable-1U"
@@
 		)
 		(embedded_fonts no)
+		(model "${KIPRJMOD}/libraries/Cherry MX.STEP"
+			(offset
+				(xyz 0 1 1.5)
+			)
+			(scale
+				(xyz 1 1 1)
+			)
+			(rotate
+				(xyz -90 -0 -0)
+			)
+		)
 	)
 	(footprint "3d:MX-Solderable-1U"
@@
 		)
 		(embedded_fonts no)
+		(model "${KIPRJMOD}/libraries/Cherry MX.STEP"
+			(offset
+				(xyz 0 1 1.5)
+			)
+			(scale
+				(xyz 1 1 1)
+			)
+			(rotate
+				(xyz -90 -0 -0)
+			)
+		)
 	)
 	(footprint "3d:MX-Solderable-1U"
@@
 		)
 		(embedded_fonts no)
+		(model "${KIPRJMOD}/libraries/Cherry MX.STEP"
+			(offset
+				(xyz 0 1 1.5)
+			)
+			(scale
+				(xyz 1 1 1)
+			)
+			(rotate
+				(xyz -90 -0 -0)
+			)
+		)
 	)
 	(footprint "pico:RPi_Pico_SMD_TH"
@@
 		)
 		(embedded_fonts no)
-		(model "C:/Users/ncara/OneDrive/IoT/Tools/KiCad/RP-Pico Libraries/Pico.wrl"
+		(model "${KIPRJMOD}/libraries/Raspberry Pi Pico-R3.STEP"
 			(offset
-				(xyz 0 0 0)
+				(xyz 0 0 3.04)
 			)
 			(scale
@@
 			)
 			(rotate
-				(xyz 0 0 0)
+				(xyz -90 -0 -0)
 			)
 		)
@@
 		)
 		(embedded_fonts no)
+		(model "${KIPRJMOD}/libraries/Cherry MX.STEP"
+			(offset
+				(xyz 0 1 1.5)
+			)
+			(scale
+				(xyz 1 1 1)
+			)
+			(rotate
+				(xyz -90 -0 -0)
+			)
+		)
 	)
 	(footprint "3d:MX-Solderable-1U"
@@
 		)
 		(embedded_fonts no)
+		(model "${KIPRJMOD}/libraries/Cherry MX.STEP"
+			(offset
+				(xyz 0 1 1.5)
+			)
+			(scale
+				(xyz 1 1 1)
+			)
+			(rotate
+				(xyz -90 -0 -0)
+			)
+		)
 	)
 	(footprint "3d:MX-Solderable-1U"
@@
 		(stroke
 			(width 0.05)
+			(type solid)
+		)
+		(fill no)
+		(layer "Edge.Cuts")
+	)
+	(gr_circle
+		(center 26.875 110.21875)
+		(end 28.575 110.21875)
+		(stroke
+			(width 0.05)
