File: big-board.kicad_sch (KiCad schematic)
At the start: 133 parts, among them SW1 SW_Push, SW10 SW_Push, SW11 SW_Push, SW12 SW_Push, SW13 SW_Push, SW14 SW_Push, SW15 SW_Push, SW16 SW_Push, SW17 SW_Push, SW18 SW_Push, SW19 SW_Push, SW2 SW_Push, SW20 SW_Push, SW21 SW_Push, SW22 SW_Push, SW23 SW_Push, SW24 SW_Push, SW25 SW_Push, SW26 SW_Push, SW27 SW_Push, SW28 SW_Push, SW29 SW_Push, SW3 SW_Push, SW30 SW_Push, SW31 SW_Push, SW32 SW_Push, SW33 SW_Push, SW34 SW_Push, SW35 SW_Push, SW36 SW_Push, SW37 SW_Push, SW38 SW_Push, SW39 SW_Push, SW4 SW_Push, SW40 SW_Push, SW41 SW_Push, SW42 SW_Push, SW43 SW_Push, SW44 SW_Push, SW45 SW_Push, SW46 SW_Push, SW47 SW_Push, SW48 SW_Push, SW49 SW_Push, SW5 SW_Push, SW50 SW_Push, SW51 SW_Push, SW52 SW_Push, SW53 SW_Push, SW54 SW_Push, SW55 SW_Push, SW56 SW_Push, SW57 SW_Push, SW58 SW_Push, SW59 SW_Push, SW6 SW_Push, SW60 SW_Push, SW61 SW_Push, SW62 SW_Push, SW63 SW_Push, SW64 SW_Push, SW65 SW_Push, SW66 SW_Push, SW7 SW_Push, SW8 SW_Push, SW9 SW_Push, U1 Pico

Commit message: start routing
Parts:
- D1, D10, D11, D12, D13, D14, D15, D16, D17, D18, D19, D2, D20, D21, D22, D23, D24, D25, D26, D27, D28, D29, D3, D30, D31, D32, D33, D34, D35, D36, D37, D38, D39, D4, D40, D41, D42, D43, D44, D45, D46, D47, D48, D49, D5, D50, D51, D52, D53, D54, D55, D56, D57, D58, D59, D6, D60, D61, D62, D63, D64, D65, D66, D7, D8, D9: footprint Diode_THT:D_DO-35_SOD27_P7.62mm_Horizontal -> Diode_THT:D_DO-35_SOD27_P2.54mm_Vertical_AnodeUp
- SW1, SW10, SW11, SW12, SW13, SW15, SW17, SW18, SW19, SW2, SW20, SW21, SW22, SW23, SW24, SW25, SW26, SW27, SW28, SW3, SW30, SW32, SW33, SW34, SW35, SW36, SW37, SW38, SW39, SW4, SW40, SW41, SW42, SW45, SW46, SW47, SW48, SW49, SW5, SW50, SW51, SW52, SW53, SW54, SW56, SW58, SW6, SW64, SW65, SW66, SW7, SW8, SW9: footprint (none) -> MX_Solderable:MX-Solderable-1U
- SW14: footprint (none) -> MX_Solderable:MX-Solderable-2U
- SW16, SW29: footprint (none) -> MX_Solderable:MX-Solderable-1.5U
- SW31: footprint (none) -> MX_Solderable:MX-Solderable-1.75U
- SW43, SW44, SW55: footprint (none) -> MX_Solderable:MX-Solderable-2.25U
- SW57, SW59, SW61, SW62, SW63: footprint (none) -> MX_Solderable:MX-Solderable-1.25U
- SW60: footprint (none) -> MX_Solderable:MX-Solderable-6.25U
- U1: footprint RPi_Pico:RPi_Pico_SMD_TH -> pico:RPi_Pico_SMD_TH
Connections:
- net GNDA: now reaches U1.33 (AGND)
- net +5V: now reaches U1.40 (VBUS)

Commit message: more pcb routing
Parts:
- D1, D10, D11, D12, D13, D14, D15, D16, D17, D18, D19, D2, D20, D21, D22, D23, D24, D25, D26, D27, D28, D29, D3, D30, D31, D32, D33, D34, D35, D36, D37, D38, D39, D4, D40, D41, D42, D43, D44, D45, D46, D47, D48, D49, D5, D50, D51, D52, D53, D54, D55, D56, D57, D58, D59, D6, D60, D61, D62, D63, D64, D65, D66, D7, D8, D9: footprint Diode_THT:D_DO-35_SOD27_P2.54mm_Vertical_AnodeUp -> Diode_THT:D_DO-35_SOD27_P7.62mm_Horizontal
Connections:
- net GND: no longer U1.13 (GND), U1.18 (GND), U1.28 (GND), U1.3 (GND), U1.38 (GND), U1.42 (GND), U1.8 (GND)
- net GNDA: no longer names the net of U1.33 (AGND)

Commit message: silkscreen stuff
Parts:
- SW1, SW10, SW11, SW12, SW13, SW15, SW17, SW18, SW19, SW2, SW20, SW21, SW22, SW23, SW24, SW25, SW26, SW27, SW28, SW3, SW30, SW32, SW33, SW34, SW35, SW36, SW37, SW38, SW39, SW4, SW40, SW41, SW42, SW45, SW46, SW47, SW48, SW49, SW5, SW50, SW51, SW52, SW53, SW54, SW56, SW58, SW6, SW64, SW65, SW66, SW7, SW8, SW9: footprint MX_Solderable:MX-Solderable-1U -> 3d:MX-Solderable-1U
Changed lines of the file:
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@@
 			)
 		)
-		(property "Footprint" "MX_Solderable:MX-Solderable-1U"
+		(property "Footprint" "3d:MX-Solderable-1U"
 			(at 224.79 35.56 0)
 			(effects
@@
 			)
 		)
-		(property "Footprint" "MX_Solderable:MX-Solderable-1U"
+		(property "Footprint" "3d:MX-Solderable-1U"
 			(at 179.07 35.56 0)
 			(effects
@@
 			)
 		)
-		(property "Footprint" "MX_Solderable:MX-Solderable-1U"
+		(property "Footprint" "3d:MX-Solderable-1U"
 			(at 194.31 35.56 0)
 			(effects
@@
 			)
 		)
-		(property "Footprint" "MX_Solderable:MX-Solderable-1U"
+		(property "Footprint" "3d:MX-Solderable-1U"
 			(at 224.79 55.88 0)
 			(effects
@@
 			)
 		)
-		(property "Footprint" "MX_Solderable:MX-Solderable-1U"
+		(property "Footprint" "3d:MX-Solderable-1U"
 			(at 163.83 35.56 0)
 			(effects
@@
 			)
 		)
-		(property "Footprint" "MX_Solderable:MX-Solderable-1U"
+		(property "Footprint" "3d:MX-Solderable-1U"
 			(at 163.83 76.2 0)
 			(effects
@@
 			)
 		)
-		(property "Footprint" "MX_Solderable:MX-Solderable-1U"
+		(property "Footprint" "3d:MX-Solderable-1U"
 			(at 118.11 35.56 0)
 			(effects
@@
 			)
 		)
-		(property "Footprint" "MX_Solderable:MX-Solderable-1U"
+		(property "Footprint" "3d:MX-Solderable-1U"
 			(at 148.59 76.2 0)
 			(effects
@@
 			)
 		)
-		(property "Footprint" "MX_Solderable:MX-Solderable-1U"
+		(property "Footprint" "3d:MX-Solderable-1U"
 			(at 255.27 35.56 0)
 			(effects
@@
 			)
 		)
-		(property "Footprint" "MX_Solderable:MX-Solderable-1U"
+		(property "Footprint" "3d:MX-Solderable-1U"
 			(at 86.36 96.52 0)
 			(effects
@@
 			)
 		)
-		(property "Footprint" "MX_Solderable:MX-Solderable-1U"
+		(property "Footprint" "3d:MX-Solderable-1U"
 			(at 54.61 35.56 0)
 			(effects
@@
 			)
 		)
-		(property "Footprint" "MX_Solderable:MX-Solderable-1U"
+		(property "Footprint" "3d:MX-Solderable-1U"
 			(at 179.07 76.2 0)
 			(effects
@@
 			)
 		)
-		(property "Footprint" "MX_Solderable:MX-Solderable-1U"
+		(property "Footprint" "3d:MX-Solderable-1U"
 			(at 163.83 55.88 0)
 			(effects
@@
 			)
 		)
-		(property "Footprint" "MX_Solderable:MX-Solderable-1U"
+		(property "Footprint" "3d:MX-Solderable-1U"
 			(at 194.31 76.2 0)
 			(effects
@@
 			)
 		)
-		(property "Footprint" "MX_Solderable:MX-Solderable-1U"
+		(property "Footprint" "3d:MX-Solderable-1U"
 			(at 194.31 96.52 0)
 			(effects
@@
 			)
 		)
-		(property "Footprint" "MX_Solderable:MX-Solderable-1U"
+		(property "Footprint" "3d:MX-Solderable-1U"
 			(at 86.36 35.56 0)
 			(effects
@@
 			)
 		)
-		(property "Footprint" "MX_Solderable:MX-Solderable-1U"
+		(property "Footprint" "3d:MX-Solderable-1U"
 			(at 118.11 76.2 0)
 			(effects
@@
 			)
 		)
-		(property "Footprint" "MX_Solderable:MX-Solderable-1U"
+		(property "Footprint" "3d:MX-Solderable-1U"
 			(at 163.83 96.52 0)
 			(effects
@@
 			)
 		)
-		(property "Footprint" "MX_Solderable:MX-Solderable-1U"
+		(property "Footprint" "3d:MX-Solderable-1U"
 			(at 209.55 55.88 0)
 			(effects
@@
 			)
 		)
-		(property "Footprint" "MX_Solderable:MX-Solderable-1U"
+		(property "Footprint" "3d:MX-Solderable-1U"
 			(at 148.59 55.88 0)
 			(effects
@@
 			)
 		)
-		(property "Footprint" "MX_Solderable:MX-Solderable-1U"
+		(property "Footprint" "3d:MX-Solderable-1U"
 			(at 148.59 96.52 0)
 			(effects
@@
 			)
 		)
-		(property "Footprint" "MX_Solderable:MX-Solderable-1U"
+		(property "Footprint" "3d:MX-Solderable-1U"
 			(at 71.12 76.2 0)
 			(effects
@@
 			)
 		)
-		(property "Footprint" "MX_Solderable:MX-Solderable-1U"
+		(property "Footprint" "3d:MX-Solderable-1U"
 			(at 148.59 35.56 0)
 			(effects
@@
 			)
 		)
-		(property "Footprint" "MX_Solderable:MX-Solderable-1U"
+		(property "Footprint" "3d:MX-Solderable-1U"
 			(at 255.27 55.88 0)
 			(effects
@@
 			)
 		)
-		(property "Footprint" "MX_Solderable:MX-Solderable-1U"
+		(property "Footprint" "3d:MX-Solderable-1U"
 			(at 102.87 35.56 0)
 			(effects
@@
 			)
 		)
-		(property "Footprint" "MX_Solderable:MX-Solderable-1U"
+		(property "Footprint" "3d:MX-Solderable-1U"
 			(at 209.55 35.56 0)
 			(effects
@@
 			)
 		)
-		(property "Footprint" "MX_Solderable:MX-Solderable-1U"
+		(property "Footprint" "3d:MX-Solderable-1U"
 			(at 118.11 96.52 0)
 			(effects
@@
 			)
 		)
-		(property "Footprint" "MX_Solderable:MX-Solderable-1U"
+		(property "Footprint" "3d:MX-Solderable-1U"
 			(at 179.07 55.88 0)
 			(effects
@@
 			)
 		)
-		(property "Footprint" "MX_Solderable:MX-Solderable-1U"
+		(property "Footprint" "3d:MX-Solderable-1U"
 			(at 71.12 55.88 0)
 			(effects
@@
 			)
 		)
-		(property "Footprint" "MX_Solderable:MX-Solderable-1U"
+		(property "Footprint" "3d:MX-Solderable-1U"
 			(at 133.35 35.56 0)
 			(effects
@@
 			)
 		)
-		(property "Footprint" "MX_Solderable:MX-Solderable-1U"
+		(property "Footprint" "3d:MX-Solderable-1U"
 			(at 54.61 76.2 0)
 			(effects
@@
 			)
 		)
-		(property "Footprint" "MX_Solderable:MX-Solderable-1U"
+		(property "Footprint" "3d:MX-Solderable-1U"
 			(at 71.12 35.56 0)
 			(effects
@@
 			)
 		)
-		(property "Footprint" "MX_Solderable:MX-Solderable-1U"
+		(property "Footprint" "3d:MX-Solderable-1U"
 			(at 179.07 118.11 0)
 			(effects
@@
 			)
 		)
-		(property "Footprint" "MX_Solderable:MX-Solderable-1U"
+		(property "Footprint" "3d:MX-Solderable-1U"
 			(at 38.1 35.56 0)
 			(effects
@@
 			)
 		)
-		(property "Footprint" "MX_Solderable:MX-Solderable-1U"
+		(property "Footprint" "3d:MX-Solderable-1U"
 			(at 133.35 55.88 0)
 			(effects
@@
 			)
 		)
-		(property "Footprint" "MX_Solderable:MX-Solderable-1U"
+		(property "Footprint" "3d:MX-Solderable-1U"
 			(at 163.83 118.11 0)
 			(effects
@@
 			)
 		)
-		(property "Footprint" "MX_Solderable:MX-Solderable-1U"
+		(property "Footprint" "3d:MX-Solderable-1U"
 			(at 102.87 76.2 0)
 			(effects
@@
 			)
 		)
-		(property "Footprint" "MX_Solderable:MX-Solderable-1U"
+		(property "Footprint" "3d:MX-Solderable-1U"
 			(at 133.35 76.2 0)
 			(effects
@@
 			)
 		)
-		(property "Footprint" "MX_Solderable:MX-Solderable-1U"
+		(property "Footprint" "3d:MX-Solderable-1U"
 			(at 54.61 118.11 0)
 			(effects
@@
 			)
 		)
-		(property "Footprint" "MX_Solderable:MX-Solderable-1U"
+		(property "Footprint" "3d:MX-Solderable-1U"
 			(at 86.36 76.2 0)
 			(effects
@@
 			)
 		)
-		(property "Footprint" "MX_Solderable:MX-Solderable-1U"
+		(property "Footprint" "3d:MX-Solderable-1U"
 			(at 118.11 55.88 0)
 			(effects
@@
 			)
 		)
-		(property "Footprint" "MX_Solderable:MX-Solderable-1U"
+		(property "Footprint" "3d:MX-Solderable-1U"
 			(at 54.61 55.88 0)
 			(effects
@@
 			)
 		)
-		(property "Footprint" "MX_Solderable:MX-Solderable-1U"
+		(property "Footprint" "3d:MX-Solderable-1U"
 			(at 71.12 96.52 0)
 			(effects
@@
 			)
 		)
-		(property "Footprint" "MX_Solderable:MX-Solderable-1U"
+		(property "Footprint" "3d:MX-Solderable-1U"
 			(at 209.55 76.2 0)
 			(effects
@@
 			)
 		)
-		(property "Footprint" "MX_Solderable:MX-Solderable-1U"
+		(property "Footprint" "3d:MX-Solderable-1U"
 			(at 179.07 96.52 0)
 			(effects
@@
 			)
 		)
-		(property "Footprint" "MX_Solderable:MX-Solderable-1U"
+		(property "Footprint" "3d:MX-Solderable-1U"
 			(at 54.61 96.52 0)
 			(effects
@@
 			)
 		)
-		(property "Footprint" "MX_Solderable:MX-Solderable-1U"
+		(property "Footprint" "3d:MX-Solderable-1U"
 			(at 102.87 55.88 0)
 			(effects
@@
 			)
 		)
-		(property "Footprint" "MX_Solderable:MX-Solderable-1U"
+		(property "Footprint" "3d:MX-Solderable-1U"
 			(at 133.35 96.52 0)
 			(effects
@@
 			)
 		)
-		(property "Footprint" "MX_Solderable:MX-Solderable-1U"
+		(property "Footprint" "3d:MX-Solderable-1U"
 			(at 86.36 55.88 0)
 			(effects
@@
 			)
 		)
-		(property "Footprint" "MX_Solderable:MX-Solderable-1U"
+		(property "Footprint" "3d:MX-Solderable-1U"
 			(at 102.87 96.52 0)
 			(effects
@@
 			)
 		)
-		(property "Footprint" "MX_Solderable:MX-Solderable-1U"
+		(property "Footprint" "3d:MX-Solderable-1U"
 			(at 194.31 55.88 0)
 			(effects
@@
 			)
 		)
-		(property "Footprint" "MX_Solderable:MX-Solderable-1U"
+		(property "Footprint" "3d:MX-Solderable-1U"
 			(at 224.79 96.52 0)
 			(effects
@@
 			)
 		)
-		(property "Footprint" "MX_Solderable:MX-Solderable-1U"
+		(property "Footprint" "3d:MX-Solderable-1U"
 			(at 148.59 118.11 0)
 			(effects

Commit message: fix pcb and generate 3d model
Connections:
- net GND: now also U1.13 (GND), U1.18 (GND), U1.28 (GND), U1.3 (GND), U1.38 (GND), U1.42 (GND), U1.8 (GND)
